File: PCB-Layout/OpenSegment-v12.sch (EAGLE design)
At the start: 46 parts, among them Q1 PNP, Q10 MMBT2222, Q11 MMBT2222, Q12 MMBT2222, Q2 PNP, Q3 PNP, Q4 PNP, Q5 PNP, Q6 PNP, Q7 PNP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

Commit message: Changing v1.2 of the PCB.
Dropped I2C jumpers. Added analog pins. Thinking about added mode select
jumpers.
Parts:
- removed R10: 10k, SparkFun:RESISTOR0402-RES
- removed SJ1, SJ2: Counter Ctl, SparkFun-Passives:SOLDERJUMPERNO
- added C1: 0.1uF, SparkFun:CAP0402-CAP
- added JP10, JP9: (no value), SparkFun-Connectors:M02PTH
Connections:
- removed net CNT-CTL: R10.1, SJ1.1, U2.ADC7
- removed net N$18: SJ2.1, U2.PB6(XTAL1/TOSC1)
- new net A6: JP9.2, U2.ADC6
- new net A7: JP10.2, U2.ADC7
- new net COUNTER: JP2.8, U2.PB6(XTAL1/TOSC1)
- new net N$11: C1.2, U2.AREF
- net GND: now also C1.1, JP10.1, JP9.1; no longer SJ1.2, SJ2.2
- net TXO: no longer JP2.8
- net VCC: no longer R10.2
Other:
- note added: "0V"
- note added: "1.59V"
- note added: "10mA"
- note added: "2.3V = R * 0.06A (60mA peak)"
- note added: "3.92V"
- note added: "4.0V"
- note added: "4.2V"
- note added: "5 - 2.1(Yellow Vf) - 0.6(NPN+PNP Vs) = 2.3V"
- note added: "5 to 12V Input"
- note added: "5.0V"
- note added: "Added A6/A7 inputs"
- note added: "Changed PB6 to dedicated counter pin"
- note added: "Changes on v1.2:"
- note added: "D22*"
- note added: "D23*"
- note added: "Measurements:"
- note added: "Removed I2C adr jumpers"
- note added: "Removed TXO connection"
- note removed: "I2C Adr"
- moved on the sheet: SJ3
