File: Hardware/OpenSegment.sch (EAGLE design)
At the start: 52 parts, among them Q1 PNP, Q10 MMBT2222, Q11 MMBT2222, Q12 MMBT2222, Q2 PNP, Q3 PNP, Q4 PNP, Q5 PNP, Q6 PNP, Q7 PNP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

Commit message: Commit For Desk Change
Only doing this commit so I can work at the new QC desk
Parts:
- added FRAME1: FRAME-LETTER, SparkFun-Aesthetics:FRAME-LETTER
- C1, C3, C4: device SparkFun:CAP0402-CAP -> SparkFun-Capacitors:0.1UF-25V(+80/-20%)(0603)
- C10: device SparkFun:CAP0402-CAP -> SparkFun-Capacitors:1.0UF-16V-10%(0603)
- R1: device SparkFun:RESISTOR0402-RES -> SparkFun-Resistors:10KOHM1/10W1%(0603)0603
- R11: device SparkFun:RESISTOR0402-RES -> SparkFun-Resistors:330OHM1/10W1%(0603)
Other:
- note added: "Revised by: Patrick Alberts"
- note added: "V14"
- moved on the sheet: Q1, Q2, Q4, Q5, Q6, Q7, Q8, R2, R3, R5, R6, R7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

Commit message: Cap/res changed, updated schematic
Changed cap/res to 0603 footprints
Updated SCH to fr-lttr  also updated to our current flag standards
Minor trace re-routing
Parts:
- R2, R3, R4, R5, R6, R7, R8, R9: device SparkFun:RESISTOR0402-RES -> SparkFun-Resistors:33OHM1/10W1%(0603)
Changed lines of the file:
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@@
 <?xml version="1.0" encoding="utf-8"?>
 <!DOCTYPE eagle SYSTEM "eagle.dtd">
-<eagle version="6.4">
+<eagle version="6.5.0">
 <drawing>
 <settings>
@@
 <part name="JP5" library="SparkFun-Electromechanical" deviceset="STAND-OFF" device=""/>
 <part name="JP6" library="SparkFun-Electromechanical" deviceset="STAND-OFF" device=""/>
-<part name="R2" library="SparkFun" deviceset="RESISTOR" device="0402-RES" value="33/68"/>
+<part name="R2" library="SparkFun-Resistors" deviceset="33OHM1/10W1%(0603)" device="" value="33/68"/>
 <part name="Q1" library="SparkFun-DiscreteSemi" deviceset="TRANSISTOR_PNP" device="SMD" value="PNP"/>
 <part name="SJ2" library="SparkFun-Passives" deviceset="SOLDERJUMPER" device="NO" value="Counter Ctl"/>
@@
 <part name="GND15" library="SparkFun" deviceset="GND" device=""/>
 <part name="JP2" library="SparkFun-Connectors" deviceset="M10" device="&quot;" value="Connections"/>
-<part name="R3" library="SparkFun" deviceset="RESISTOR" device="0402-RES" value="33/68"/>
-<part name="R4" library="SparkFun" deviceset="RESISTOR" device="0402-RES" value="33/68"/>
-<part name="R5" library="SparkFun" deviceset="RESISTOR" device="0402-RES" value="33/68"/>
-<part name="R6" library="SparkFun" deviceset="RESISTOR" device="0402-RES" value="33/68"/>
-<part name="R7" library="SparkFun" deviceset="RESISTOR" device="0402-RES" value="33/68"/>
-<part name="R8" library="SparkFun" deviceset="RESISTOR" device="0402-RES" value="33/68"/>
-<part name="R9" library="SparkFun" deviceset="RESISTOR" device="0402-RES" value="33/68"/>
+<part name="R3" library="SparkFun-Resistors" deviceset="33OHM1/10W1%(0603)" device="" value="33/68"/>
+<part name="R4" library="SparkFun-Resistors" deviceset="33OHM1/10W1%(0603)" device="" value="33/68"/>
+<part name="R5" library="SparkFun-Resistors" deviceset="33OHM1/10W1%(0603)" device="" value="33/68"/>
+<part name="R6" library="SparkFun-Resistors" deviceset="33OHM1/10W1%(0603)" device="" value="33/68"/>
+<part name="R7" library="SparkFun-Resistors" deviceset="33OHM1/10W1%(0603)" device="" value="33/68"/>
+<part name="R8" library="SparkFun-Resistors" deviceset="33OHM1/10W1%(0603)" device="" value="33/68"/>
+<part name="R9" library="SparkFun-Resistors" deviceset="33OHM1/10W1%(0603)" device="" value="33/68"/>
 <part name="GND16" library="SparkFun" deviceset="GND" device=""/>
 <part name="U$2" library="SparkFun" deviceset="LOGO-SFE" device="SK"/>

Commit message: Desk Change
Parts:
- removed U$3: CREATIVE_COMMONS, SparkFun:CREATIVE_COMMONS
- FRAME1: value FRAME-LETTER -> FRAME-LEDGER; device SparkFun-Aesthetics:FRAME-LETTER -> SparkFun-Aesthetics:FRAME-LEDGER
- LED1: device SparkFun:LED0603 -> SparkFun-LED:LED-RED0603
Other:
- note added: "Revision History"
- moved on the sheet: C1, C10, C13, C19, C3, C4, JP1, JP10, JP11, JP12, JP13, JP2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

Commit message: SCH cleanup
Sch clean up as well as new symbols for the transistors.
Parts:
- Q1, Q2, Q3, Q4, Q5, Q6, Q7, Q8: device SparkFun-DiscreteSemi:TRANSISTOR_PNPSMD -> SparkFun-DiscreteSemi:TRANSISTOR-PNP-DDTB142TC
- Q10, Q11, Q12, Q9: device SparkFun-DiscreteSemi:TRANSISTOR_NPNSOT23-3 -> SparkFun-DiscreteSemi:TRANSISTOR-NPN-DDTD142TC
Other:
- note removed: "1 for counter"
- note removed: "12 for Display"
- note removed: "2 for I2C"
- note removed: "2 for I2C Address"
- note removed: "2 for Serial"
- note removed: "2.3V = R * 0.06A (60mA peak)"
- note removed: "4 / 0.08 = 50Ohm"
- note removed: "4 for SPI"
- note removed: "5 - 1 = 4V"
- note removed: "5 - 2.1(Yellow Vf) - 0.6(NPN+PNP Vs) = 2.3V"
- note removed: "80mA Max @ 25% Duty cycle"
- note removed: "Add OSHW logo"
- note removed: "Add reset breakout"
- note removed: "Add silk to top side A6/7"
- note removed: "Added A6/A7 inputs"
- note removed: "Added mode jumpers"
- note removed: "Changed SPI pins to SDO/SDI to match"
- note removed: "Changes on v1.1:"
- note removed: "Changes on v1.2:"
- note removed: "Changes on v1.3:"
- note removed: "Fixed 7-seg footprint"
- note removed: "Fixed silk"
- note removed: "Ganged I2C + pwr"
- note removed: "Measurements show 10mA. Changing to 27 Ohm"
- note removed: "Move in 10uF cap"
- note removed: "R = 38.3 Ohm"
- note removed: "Removed I2C adr jumpers"
- note removed: "Revision History"
- note removed: "Silkscreen squares for colors"
- note removed: "Swapped NPN/PNPs"
- note removed: "original S7S"
- note removed: "v1.0"
- moved on the sheet: C10, C13, C19, C4, JP10, JP11, JP12, JP13, JP2, JP9, LED1, R11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

Commit message: added regular fiducials
Parts:
- removed JP14, JP7: FIDUCIALUFIDUCIAL, SparkFun:FIDUCIALUFIDUCIAL
- added FID1, FID2: FIDUCIAL1X2, SparkFun-Aesthetics:FIDUCIAL1X2
Changed lines of the file:
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@@
 <?xml version="1.0" encoding="utf-8"?>
 <!DOCTYPE eagle SYSTEM "eagle.dtd">
-<eagle version="6.4">
+<eagle version="6.5.0">
 <drawing>
 <settings>
@@
 <part name="JP12" library="SparkFun-Connectors" deviceset="M02" device="PTH"/>
 <part name="JP13" library="SparkFun-Connectors" deviceset="M02" device="PTH"/>
-<part name="JP7" library="SparkFun" deviceset="FIDUCIAL" device="UFIDUCIAL"/>
-<part name="JP14" library="SparkFun" deviceset="FIDUCIAL" device="UFIDUCIAL"/>
+<part name="FID1" library="SparkFun-Aesthetics" deviceset="FIDUCIAL" device="1X2"/>
+<part name="FID2" library="SparkFun-Aesthetics" deviceset="FIDUCIAL" device="1X2"/>
 </parts>
 <sheets>
@@
 <instance part="JP12" gate="G$1" x="218.44" y="48.26"/>
 <instance part="JP13" gate="G$1" x="218.44" y="33.02"/>
-<instance part="JP7" gate="G$1" x="424.18" y="30.48"/>
-<instance part="JP14" gate="G$1" x="424.18" y="25.4"/>
+<instance part="FID1" gate="G$1" x="429.26" y="33.02"/>
+<instance part="FID2" gate="G$1" x="429.26" y="25.4"/>
 </instances>
 <busses>
